File: Hardware/2-Layer-Version/Blueberry Pi.brd (EAGLE design)
At the start: 99.1 x 64.8 mm, 172 parts, among them IC3 AT45DB161D, J1 TRANSFLASH-LOCK, J2 AUDIO_JACK_SMD, Q1 24Mhz, Q2 32kHz, X1 USB-B-S, X3 52745-2290

Commit message: new version
Parts:
- removed ANT1: (no value), rcl:R1206
- removed IC3: AT45DB161D, SparkFun-Retired:SO08-EIAJ
- removed R46: 10k, rcl:R0603
- added ANT2: U-FL, Seeed-Connector:U-FL3P-SMD-2.6X2.6X1.0MM
- added R3: 10M, rcl:R0603
- added R4: 0R, rcl:R0603
- added U1: 25F32006WSOI, SparkFun-IC-Memory:SO08-EIAJ
- C4: value 1µF -> 33pF
- C5, C6: value 1µF -> 10µF; device rcl:C0603 -> rcl:C0805
- L5: value 2,2µH -> 2.2µH
- R47: value (none) -> 5,1
- U$5: device con-hirose:ZX62R-B-5P -> Blueberry Pi:CON-HIROSE_ZX62R-B-5P
- moved C45 20.1 mm to (65.0, 13.2), turned to 180 degrees
- moved L5 18.0 mm to (69.3, 14.4), turned to 180 degrees
- moved C46 17.4 mm to (69.3, 10.6)
- moved R54 17.4 mm to (70.7, 3.47), turned to 90 degrees
- moved R57 17.2 mm to (65.0, 10.6), turned to 180 degrees
- moved C40 15.7 mm to (69.4, 8.47), turned to 0 degrees
- moved R58 15.3 mm to (65.0, 8.23), turned to 180 degrees
- moved C5 14.4 mm to (55.3, 10.7), flipped to the bottom, turned to 180 degrees
- moved C43 14.3 mm to (85.0, 13.4), turned to 90 degrees
- moved R7 13.9 mm to (72.9, 3.45), turned to 90 degrees
- moved C44 13.2 mm to (83.0, 2.78), turned to 270 degrees
- moved C42 12.6 mm to (77.6, 14.3), turned to 270 degrees
- moved C41 11.1 mm to (75.1, 3.44), turned to 90 degrees
- moved R56 10.9 mm to (73.0, 14.3), turned to 270 degrees
- moved L3 9.82 mm to (78.8, 2.88), turned to 90 degrees
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Connections:
- removed net N$61: JP7.1, U$2.P$44
- removed net N$63: JP7.3, U$2.P$42
- removed net N$9 (its old number): R46.1, U$9.4
- new net N$11: JP7.1, U$2.P$42
- new net N$2: ANT2.D, C4.2
- new net N$5: JP7.3, U$2.P$44
- net +3V3: now also C5.1, C6.1, JP6.17, R8.2, U1.3, U1.7, U1.8; no longer IC3.3, IC3.5, IC3.6, R8.1
- net +5V: now also R4.2, U$9.4, X1.VBUS; no longer X1.VUSB
- net CSI_D0/LCD_D2: no longer JP10.20, JP6.16
- net CSI_D1/LCD_D3: no longer JP10.19, JP6.15
- net CSI_D10/LCD_D14: now also JP10.10, JP6.10
- net CSI_D11/LCD_D15: now also JP10.9, JP6.9
- net CSI_D2/LCD_D4: now also JP10.20; no longer JP10.16, JP6.14
- net CSI_D3/LCD_D5: now also JP10.19; no longer JP10.15, JP6.13
- net CSI_D4/LCD_D6: now also JP10.16, JP6.16; no longer JP10.14, JP6.12
- net CSI_D5/LCD_D7: now also JP10.15, JP6.15; no longer JP10.13, JP6.11
- net CSI_D6/LCD_D10: now also JP10.14, JP6.14; no longer JP10.12, JP6.10
- net CSI_D7/LCD_D11: now also JP10.13, JP6.13; no longer JP10.11, JP6.9
- net CSI_D8/LCD_D12: now also JP10.12, JP6.12; no longer JP10.10
- net CSI_D9/LCD_D13: now also JP10.11, JP6.11; no longer JP10.9
- net GND: now also ANT2.GND1, ANT2.GND2, U1.4; no longer ANT1.1, IC3.7, JP6.17, R46.2
- net N$13: no longer C5.1
- net N$14: now also J3.35, R4.1; no longer ANT1.2, C4.2, C6.1
- net N$29: now also R3.1
- net N$30: now also R3.2
- net SPI1/CS: now also R8.1, U1.1; no longer IC3.4, R8.2
- net SPI1/MISO: now also U1.2; no longer IC3.8
- net SPI1/MOSI: now also U1.5; no longer IC3.1
- net SPI1/SCK: now also U1.6; no longer IC3.2
Routing:
- net CSI_D10/LCD_D14: track 51.6 -> 103.8 mm, vias 1 -> 4
- net CSI_D0/LCD_D2: track 90.6 -> 40.5 mm, vias 4 -> 3
- net CSI_D11/LCD_D15: track 52.7 -> 99.6 mm, vias 1 -> 3
- net CSI_D1/LCD_D3: track 90.1 -> 45.5 mm, vias 3 -> 2
- net N$5: track 0.00 -> 33.8 mm
- net N$63: track 27.8 -> 0.00 mm, vias 2 -> 0
- net N$11: track 0.00 -> 27.4 mm
- net N$61: track 24.9 -> 0.00 mm, vias 1 -> 0
- net +1V2: track 157.9 -> 176.8 mm, vias 10 -> 9
- net +5V: track 284.0 -> 301.5 mm, vias 13 -> 16
- net CSI_D8/LCD_D12: track 93.7 -> 106.6 mm
- net +3V3: track 485.3 -> 475.0 mm, vias 30 -> 31
- net CSI_D3/LCD_D5: track 86.9 -> 96.5 mm
- net +3V3A: track 114.4 -> 124.0 mm
- net N$71: track 7.54 -> 16.3 mm, vias 0 -> 2
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