File: Hardware/2-Layer-Version/Blueberry Pi.sch (EAGLE design)
At the start: 172 parts, among them IC3 AT45DB161D, J1 TRANSFLASH-LOCK, J2 AUDIO_JACK_SMD, J3 40PINFPCH15-1LW, Q1 24Mhz, Q2 32kHz, X1 USB-B-S, X3 52745-2290

Commit message: new version
Parts:
- removed ANT1: (no value), rcl:R-EU_R1206
- removed IC3: AT45DB161D, SparkFun-Retired:AT45DB161D
- removed R46: 10k, rcl:R-EU_R0603
- added ANT2: U-FL, Seeed-Connector:ANTENNA-CONN-U-FL(3P)
- added R3: 10M, rcl:R-EU_R0603
- added R4: 0R, rcl:R-EU_R0603
- added U1: 25F32006WSOI, SparkFun-IC-Memory:SPI_FLASH-X25XXSMD1
- C4: value 1µF -> 33pF
- C5, C6: value 1µF -> 10µF; device rcl:C-EUC0603 -> rcl:C-EUC0805
- L5: value 2,2µH -> 2.2µH
- R47: value (none) -> 5,1
- U$5: value MICRO-USB-SHIELD-ZX62R-B-5P -> CON-HIROSE_MICRO-USB-SHIELD-ZX62R-B-5P; device con-hirose:MICRO-USB-SHIELD-ZX62R-B-5P -> Blueberry Pi:CON-HIROSE_MICRO-USB-SHIELD-ZX62R-B-5P
Connections:
- removed net N$61: JP7.1, U$2.UART_CTS
- removed net N$63: JP7.3, U$2.UART_TXD
- removed net N$9 (its old number): R46.1, U$9.EN
- new net N$11: JP7.1, U$2.UART_TXD
- new net N$2: ANT2.D, C4.2
- new net N$5: JP7.3, U$2.UART_CTS
- net +3V3: now also C5.1, C6.1, JP6.17, R8.2, U1.HOLD, U1.VCC, U1.WP; no longer IC3.RST, IC3.VCC, IC3.WP, R8.1
- net +5V: now also R4.2, U$9.EN
- net CSI_D0/LCD_D2: no longer JP10.20, JP6.16
- net CSI_D1/LCD_D3: no longer JP10.19, JP6.15
- net CSI_D10/LCD_D14: now also JP10.10, JP6.10
- net CSI_D11/LCD_D15: now also JP10.9, JP6.9
- net CSI_D2/LCD_D4: now also JP10.20; no longer JP10.16, JP6.14
- net CSI_D3/LCD_D5: now also JP10.19; no longer JP10.15, JP6.13
- net CSI_D4/LCD_D6: now also JP10.16, JP6.16; no longer JP10.14, JP6.12
- net CSI_D5/LCD_D7: now also JP10.15, JP6.15; no longer JP10.13, JP6.11
- net CSI_D6/LCD_D10: now also JP10.14, JP6.14; no longer JP10.12, JP6.10
- net CSI_D7/LCD_D11: now also JP10.13, JP6.13; no longer JP10.11, JP6.9
- net CSI_D8/LCD_D12: now also JP10.12, JP6.12; no longer JP10.10
- net CSI_D9/LCD_D13: now also JP10.11, JP6.11; no longer JP10.9
- net GND: now also ANT2.GND1, ANT2.GND2, U1.GND; no longer ANT1.1, IC3.GND, JP6.17, R46.2
- net N$13: no longer C5.1
- net N$14: now also J3-35.MS, R4.1; no longer ANT1.2, C4.2, C6.1
- net N$29: now also R3.1
- net N$30: now also R3.2
- net SPI1/CS: now also R8.1, U1.CS; no longer IC3.CS, R8.2
- net SPI1/MISO: now also U1.MISO; no longer IC3.SO
- net SPI1/MOSI: now also U1.MOSI; no longer IC3.SI
- net SPI1/SCK: now also U1.SCK; no longer IC3.SCK
Other:
- note added: "Connect VCC-PE to 1-8V - 3,3V, otherwise the V3s won't boot."
- note added: "Connect VCC-RTC to 3,3V or a battery, otherwise the V3s won't boot."
- note added: "only mount R4 if you want to have 5V on the 40 pin FFC (Expansion)"
- moved on the sheet: C1, C32, C33, C35, C4, C40, C41, C42, C43, C44, C45, C46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
